Commit message: updated cartographer

File: cartographer_ros/urdf/os1_sensor.urdf (robot description, URDF)
Before this commit: robot cartographer_backpack_3d, 3 links, 2 joints
Links:
- added link os1_lidar; visual cylinder length=0.07 radius=0.05
- added link os1_sensor
- link os1: geometry 
Joints:
- added joint os1_link_joint_legacy: type fixed, parent base_link, child os1, origin xyz=0.00 0. 0.03618 rpy=0. 0 0
- added joint sensor_link_joint: type fixed, parent base_link, child os1_sensor, origin xyz=0 0 0 rpy=0 0 0
- joint imu_link_joint: origin xyz=0 0 0 rpy=0 0 0 -> xyz=0.006253 -0.011775 0.007645 rpy=0 0 0; parent base_link -> os1_sensor
- joint os1_link_joint: child os1 -> os1_lidar; origin xyz=0.00 0. 0.0 rpy=0. 0 0 -> xyz=0.0 0.0 0.03618 rpy=0 0 3.14159; parent base_link -> os1_sensor

File: ouster_description/urdf/OS1-64.urdf.xacro (robot description, xacro)
@@ -41,5 +41,5 @@
       <parent link="${name}" />
       <child link="os1_lidar" />
-      <origin xyz="0.0 0.0 0.03618" rpy="0 0 3.14159" />
+      <origin xyz="0.0 0.0 0.03618" rpy="0 0 0" />
     </joint>
     <!-- Gazebo requires the ouster_gazebo_plugins package -->
