Commit message: updated gazebo plugin

File: ouster_description/urdf/OS1-64.urdf.xacro (robot description, xacro)
@@ -2,5 +2,5 @@
 <robot xmlns:xacro="http://www.ros.org/wiki/xacro" name="OS1-64">
   <xacro:property name="M_PI" value="3.1415926535897931" />
-  <xacro:macro name="OS1-64" params="*origin parent:=base_link name:=ouster topic:=/points hz:=10 lasers:=64 samples:=512 min_range:=0.9 max_range:=75.0 noise:=0.008 min_angle:=-${M_PI} max_angle:=${M_PI}">
+  <xacro:macro name="OS1-64" params="*origin parent:=base_link name:=os1 topic:=/os1_cloud_node/points hz:=10 lasers:=64 samples:=512 min_range:=0.9 max_range:=75.0 noise:=0.008 min_angle:=-${M_PI} max_angle:=${M_PI}">
     <joint name="${name}_base_mount_joint" type="fixed">
       <xacro:insert_block name="origin" />

Commit message: updated tf frames and added IMU

File: ouster_description/urdf/OS1-64.urdf.xacro (robot description, xacro)
@@ -2,6 +2,6 @@
 <robot xmlns:xacro="http://www.ros.org/wiki/xacro" name="OS1-64">
   <xacro:property name="M_PI" value="3.1415926535897931" />
-  <xacro:macro name="OS1-64" params="*origin parent:=base_link name:=os1 topic:=/os1_cloud_node/points hz:=10 lasers:=64 samples:=512 min_range:=0.9 max_range:=75.0 noise:=0.008 min_angle:=-${M_PI} max_angle:=${M_PI}">
-    <joint name="${name}_base_mount_joint" type="fixed">
+  <xacro:macro name="OS1-64" params="*origin parent:=base_link name:=os1_sensor topic:=/os1_cloud_node/points hz:=10 lasers:=64 samples:=512 min_range:=0.9 max_range:=75.0 noise:=0.008 min_angle:=-${M_PI} max_angle:=${M_PI}">
+    <joint name="mount_joint" type="fixed">
       <xacro:insert_block name="origin" />
       <parent link="${parent}"/>
@@ -18,14 +18,29 @@
          <origin xyz="0 0 0.0365" rpy="0 0 0" />
          <geometry>
- 	   <cylinder radius="0.04" length="0.073"/>
+ 	        <cylinder radius="0.04" length="0.073"/>
          </geometry>
       </collision>
       <visual name="base_visual">
-         <origin xyz="0 0 0" rpy="0 0 1.5707" />
+         <origin xyz="0 0 0.0" rpy="0 0 1.5707" />
          <geometry>
-	    <mesh filename="package://ouster_description/meshes/os1_64.dae" />
+	         <mesh filename="package://ouster_description/meshes/os1_64.dae" />
+           <!-- <cylinder length="0.073" radius="0.04" /> -->
          </geometry>
       </visual>
-   </link>
+    </link>
+    <link name="os1_imu" />
+    <link name="os1_lidar" />
+    <joint name="imu_link_joint" type="fixed">
+      <parent link="${name}" />
+      <child link="os1_imu" />
+      <origin xyz="0.006253 -0.011775 0.007645" rpy="0 0 0" />
+    </joint>
+    <gazebo reference="os1_imu">
+    </gazebo>
+    <joint name="lidar_link_joint" type="fixed">
+      <parent link="${name}" />
+      <child link="os1_lidar" />
+      <origin xyz="0.0 0.0 0.03618" rpy="0 0 3.14159" />
+    </joint>
     <!-- Gazebo requires the ouster_gazebo_plugins package -->
     <gazebo reference="${name}">
@@ -34,33 +49,7 @@
           <visualize>false</visualize>
           <update_rate>${hz}</update_rate>
-          <ray>
-            <scan>
-              <horizontal>
-                <samples>${samples}</samples>
-                <resolution>1</resolution>
-                <min_angle>${min_angle}</min_angle>
-                <max_angle>${max_angle}</max_angle>
-              </horizontal>
-              <vertical>
-                <samples>${lasers}</samples>
-                <resolution>1</resolution>
-                <min_angle>-${15*M_PI/180.0}</min_angle>
-                <max_angle>${15*M_PI/180.0}</max_angle>
-              </vertical>
-            </scan>
-            <range>
-              <min>${min_range}</min>
-              <max>${max_range}</max>
-              <resolution>0.03</resolution>
-            </range>
-            <noise>
-              <type>gaussian</type>
-              <mean>0.0</mean>
-              <stddev>0.0</stddev>
-            </noise>
-          </ray>
           <plugin name="gazebo_ros_laser_controller" filename="libgazebo_ros_ouster_laser.so">
             <topicName>${topic}</topicName>
-            <frameName>${name}</frameName>
+            <frameName>os1_lidar</frameName>
             <min_range>${min_range}</min_range>
             <max_range>${max_range}</max_range>
@@ -69,4 +58,19 @@
         </sensor>
     </gazebo>
+    <!-- IMU -->
+  <gazebo>
+    <plugin name="imu_controller" filename="libhector_gazebo_ros_imu.so">
+      <robotNamespace>/</robotNamespace>
+      <updateRate>200.0</updateRate>
+      <bodyName>os1_imu</bodyName>
+      <topicName>/os1_cloud_node/imu</topicName>
+      <accelDrift>0.005 0.005 0.005</accelDrift>
+      <accelGaussianNoise>0.005 0.005 0.005</accelGaussianNoise>
+      <rateDrift>0.005 0.005 0.005 </rateDrift>
+      <rateGaussianNoise>0.005 0.005 0.005 </rateGaussianNoise>
+      <headingDrift>0.005</headingDrift>
+      <headingGaussianNoise>0.005</headingGaussianNoise>
+    </plugin>
+  </gazebo>
   </xacro:macro>
 </robot>

File: ouster_description/urdf/example.urdf.xacro (robot description, xacro)
@@ -1,4 +1,4 @@
 <?xml version="1.0"?>
-<robot xmlns:xacro="http://www.ros.org/wiki/xacro" name="example">
+<robot xmlns:xacro="http://www.ros.org/wiki/xacro" name="os1_example">
   <!-- Base Footprint -->
   <link name="base_footprint" />
@@ -30,5 +30,5 @@
 -
   <xacro:include filename="$(find ouster_description)/urdf/OS1-64.urdf.xacro"/>
-  <OS1-64 parent="base_link" name="ouster" topic="/points" hz="10" samples="220">
+  <OS1-64 parent="base_link" name="os1_sensor" hz="10" samples="220">
     <origin xyz="0 0 1.2" rpy="0 0 0" />
   </OS1-64>

Commit message: added os1 arguments

File: ouster_description/urdf/OS1-64.urdf.xacro (robot description, xacro)
@@ -2,6 +2,6 @@
 <robot xmlns:xacro="http://www.ros.org/wiki/xacro" name="OS1-64">
   <xacro:property name="M_PI" value="3.1415926535897931" />
-  <xacro:macro name="OS1-64" params="*origin parent:=base_link name:=os1_sensor topic:=/os1_cloud_node/points hz:=10 lasers:=64 samples:=512 min_range:=0.9 max_range:=75.0 noise:=0.008 min_angle:=-${M_PI} max_angle:=${M_PI}">
-    <joint name="mount_joint" type="fixed">
+  <xacro:macro name="OS1-64" params="*origin parent:=base_link name:=os1_sensor topic_points:=/os1_cloud_node/points topic_imu:=/os1_cloud_node/imu hz:=10 lasers:=64 samples:=512 min_range:=0.9 max_range:=75.0 noise:=0.008 min_angle:=-${M_PI} max_angle:=${M_PI} lidar_link:=os1_lidar imu_link:=os1_imu vfov_min:=-.26 vfov_max:=.26">
+    <joint name="${name}_mount_joint" type="fixed">
       <xacro:insert_block name="origin" />
       <parent link="${parent}"/>
@@ -29,16 +29,16 @@
       </visual>
     </link>
-    <link name="os1_imu" />
-    <link name="os1_lidar" />
-    <joint name="imu_link_joint" type="fixed">
+    <link name="${imu_link}" />
+    <link name="${lidar_link}" />
+    <joint name="${name}_imu_link_joint" type="fixed">
       <parent link="${name}" />
-      <child link="os1_imu" />
+      <child link="${imu_link}" />
       <origin xyz="0.006253 -0.011775 0.007645" rpy="0 0 0" />
     </joint>
-    <gazebo reference="os1_imu">
+    <gazebo reference="${imu_link}">
     </gazebo>
-    <joint name="lidar_link_joint" type="fixed">
+    <joint name="${name}_lidar_link_joint" type="fixed">
       <parent link="${name}" />
-      <child link="os1_lidar" />
+      <child link="${lidar_link}" />
       <origin xyz="0.0 0.0 0.03618" rpy="0 0 0" />
     </joint>
@@ -60,6 +60,6 @@
                 <samples>${lasers}</samples>
                 <resolution>1</resolution>
-                <min_angle>-${15*M_PI/180.0}</min_angle>
-                <max_angle>${15*M_PI/180.0}</max_angle>
+                <min_angle>${vfov_min}</min_angle>
+                <max_angle>${vfov_max}</max_angle>
               </vertical>
             </scan>
@@ -71,6 +71,6 @@
           </ray>
           <plugin name="gazebo_ros_laser_controller" filename="libgazebo_ros_ouster_laser.so">
-            <topicName>${topic}</topicName>
-            <frameName>os1_lidar</frameName>
+            <topicName>${topic_points}</topicName>
+            <frameName>${lidar_link}</frameName>
             <min_range>${min_range}</min_range>
             <max_range>${max_range}</max_range>
@@ -84,6 +84,6 @@
       <robotNamespace>/</robotNamespace>
       <updateRate>100.0</updateRate>
-      <bodyName>os1_imu</bodyName>
-      <topicName>/os1_cloud_node/imu</topicName>
+      <bodyName>${imu_link}</bodyName>
+      <topicName>${topic_imu}</topicName>
       <accelDrift>0.005 0.005 0.005</accelDrift>
       <accelGaussianNoise>0.005 0.005 0.005</accelGaussianNoise>

File: ouster_description/urdf/example.urdf.xacro (robot description, xacro)
@@ -28,5 +28,4 @@
     </inertial>
   </link>
--
   <xacro:include filename="$(find ouster_description)/urdf/OS1-64.urdf.xacro"/>
   <OS1-64 parent="base_link" name="os1_sensor" hz="10" samples="220">
